Commit message: add scale property to support re-scaling
following the size of gripper that generated from Fusion360, this size of robot seems bigger than real robot.

File: denso_cobotta_descriptions/cobotta_description/cobotta.urdf.xacro (robot description, xacro)
@@ -6,4 +6,5 @@
 		NOTE: These are roughly estimated values.
 	-->
+	<xacro:property name="scale" value ="0.8" />
 	<xacro:property name="joint_damping" value="0.001" />
 	<xacro:property name="joint_friction" value="0.61" />
@@ -42,11 +43,11 @@
 			<origin rpy="0 0 0" xyz="0 0 0"/>
 			<geometry>
-				<mesh filename="package://denso_cobotta_descriptions/cobotta_description/base_link.dae" scale="1 1 1"/>
-			</geometry>
-		</visual>
-		<collision>
-			<origin rpy="0 0 0" xyz="0 0 0"/>
-			<geometry>
-				<mesh filename="package://denso_cobotta_descriptions/cobotta_description/base_link.dae" scale="1 1 1"/>
+				<mesh filename="package://denso_cobotta_descriptions/cobotta_description/base_link.dae" scale="${scale} ${scale} ${scale}"/>
+			</geometry>
+		</visual>
+		<collision>
+			<origin rpy="0 0 0" xyz="0 0 0"/>
+			<geometry>
+				<mesh filename="package://denso_cobotta_descriptions/cobotta_description/base_link.dae" scale="${scale} ${scale} ${scale}"/>
 			</geometry>
 		</collision>
@@ -59,11 +60,11 @@
 			<origin rpy="0 0 0" xyz="0 0 0"/>
 			<geometry>
-				<mesh filename="package://denso_cobotta_descriptions/cobotta_description/J1.dae" scale="1 1 1"/>
-			</geometry>
-		</visual>
-		<collision>
-			<origin rpy="0 0 0" xyz="0 0 0"/>
-			<geometry>
-				<mesh filename="package://denso_cobotta_descriptions/cobotta_description/J1.dae" scale="1 1 1"/>
+				<mesh filename="package://denso_cobotta_descriptions/cobotta_description/J1.dae" scale="${scale} ${scale} ${scale}"/>
+			</geometry>
+		</visual>
+		<collision>
+			<origin rpy="0 0 0" xyz="0 0 0"/>
+			<geometry>
+				<mesh filename="package://denso_cobotta_descriptions/cobotta_description/J1.dae" scale="${scale} ${scale} ${scale}"/>
 			</geometry>
 		</collision>
@@ -94,11 +95,11 @@
 			<origin rpy="0 0 0" xyz="0 0 0"/>
 			<geometry>
-				<mesh filename="package://denso_cobotta_descriptions/cobotta_description/J2.dae" scale="1 1 1"/>
-			</geometry>
-		</visual>
-		<collision>
-			<origin rpy="0 0 0" xyz="0 0 0"/>
-			<geometry>
-				<mesh filename="package://denso_cobotta_descriptions/cobotta_description/J2.dae" scale="1 1 1"/>
+				<mesh filename="package://denso_cobotta_descriptions/cobotta_description/J2.dae" scale="${scale} ${scale} ${scale}"/>
+			</geometry>
+		</visual>
+		<collision>
+			<origin rpy="0 0 0" xyz="0 0 0"/>
+			<geometry>
+				<mesh filename="package://denso_cobotta_descriptions/cobotta_description/J2.dae" scale="${scale} ${scale} ${scale}"/>
 			</geometry>
 		</collision>
@@ -110,5 +111,5 @@
 		<parent link="J1"/>
 		<child link="J2"/>
-		<origin rpy="0.000000 0.000000 0.000000" xyz="0.000000 0.000000 0.180000" />
+		<origin rpy="0.000000 0.000000 0.000000" xyz="0.000000 0.000000 ${0.180000*scale}" />
 		<axis xyz="-0.000000 1.000000 -0.000000" />
 		<limit effort="10" lower="-1.047198" upper="1.745329" velocity="0.392175482923126" />
@@ -129,11 +130,11 @@
 			<origin rpy="0 0 0" xyz="0 0 0"/>
 			<geometry>
-				<mesh filename="package://denso_cobotta_descriptions/cobotta_description/J3.dae" scale="1 1 1"/>
-			</geometry>
-		</visual>
-		<collision>
-			<origin rpy="0 0 0" xyz="0 0 0"/>
-			<geometry>
-				<mesh filename="package://denso_cobotta_descriptions/cobotta_description/J3.dae" scale="1 1 1"/>
+				<mesh filename="package://denso_cobotta_descriptions/cobotta_description/J3.dae" scale="${scale} ${scale} ${scale}"/>
+			</geometry>
+		</visual>
+		<collision>
+			<origin rpy="0 0 0" xyz="0 0 0"/>
+			<geometry>
+				<mesh filename="package://denso_cobotta_descriptions/cobotta_description/J3.dae" scale="${scale} ${scale} ${scale}"/>
 			</geometry>
 		</collision>
@@ -145,5 +146,5 @@
 		<parent link="J2"/>
 		<child link="J3"/>
-		<origin rpy="0.000000 0.000000 0.000000" xyz="0.000000 0.000000 0.165000" />
+		<origin rpy="0.000000 0.000000 0.000000" xyz="0.000000 0.000000 ${0.165000*scale}" />
 		<axis xyz="-0.000000 1.000000 -0.000000" />
 		<limit effort="10" lower="0.3141593" upper="2.443461" velocity="0.725707902979242" />
@@ -164,11 +165,11 @@
 			<origin rpy="0 0 0" xyz="0 0 0"/>
 			<geometry>
-				<mesh filename="package://denso_cobotta_descriptions/cobotta_description/J4.dae" scale="1 1 1"/>
-			</geometry>
-		</visual>
-		<collision>
-			<origin rpy="0 0 0" xyz="0 0 0"/>
-			<geometry>
-				<mesh filename="package://denso_cobotta_descriptions/cobotta_description/J4.dae" scale="1 1 1"/>
+				<mesh filename="package://denso_cobotta_descriptions/cobotta_description/J4.dae" scale="${scale} ${scale} ${scale}"/>
+			</geometry>
+		</visual>
+		<collision>
+			<origin rpy="0 0 0" xyz="0 0 0"/>
+			<geometry>
+				<mesh filename="package://denso_cobotta_descriptions/cobotta_description/J4.dae" scale="${scale} ${scale} ${scale}"/>
 			</geometry>
 		</collision>
@@ -180,5 +181,5 @@
 		<parent link="J3"/>
 		<child link="J4"/>
-		<origin rpy="0.000000 0.000000 0.000000" xyz="-0.012000 0.020000 0.088000" />
+		<origin rpy="0.000000 0.000000 0.000000" xyz="${-0.012000*scale} ${0.020000*scale} ${0.088000*scale}" />
 		<axis xyz="-0.000000 -0.000000 1.000000" />
 		<limit effort="10" lower="-2.96706" upper="2.96706" velocity="0.739146938219599" />
@@ -199,11 +200,11 @@
 			<origin rpy="0 0 0" xyz="0 0 0"/>
 			<geometry>
-				<mesh filename="package://denso_cobotta_descriptions/cobotta_description/J5.dae" scale="1 1 1"/>
-			</geometry>
-		</visual>
-		<collision>
-			<origin rpy="0 0 0" xyz="0 0 0"/>
-			<geometry>
-				<mesh filename="package://denso_cobotta_descriptions/cobotta_description/J5.dae" scale="1 1 1"/>
+				<mesh filename="package://denso_cobotta_descriptions/cobotta_description/J5.dae" scale="${scale} ${scale} ${scale}"/>
+			</geometry>
+		</visual>
+		<collision>
+			<origin rpy="0 0 0" xyz="0 0 0"/>
+			<geometry>
+				<mesh filename="package://denso_cobotta_descriptions/cobotta_description/J5.dae" scale="${scale} ${scale} ${scale}"/>
 			</geometry>
 		</collision>
@@ -215,5 +216,5 @@
 		<parent link="J4"/>
 		<child link="J5"/>
-		<origin rpy="0.000000 0.000000 0.000000" xyz="0.000000 -0.020000 0.089500" />
+		<origin rpy="0.000000 0.000000 0.000000" xyz="0.000000 ${-0.020000*scale} ${0.089500*scale}" />
 		<axis xyz="-0.000000 1.000000 -0.000000" />
 		<limit effort="10" lower="-1.658063" upper="2.356194" velocity="0.739146938219599" />
@@ -234,11 +235,11 @@
 			<origin rpy="0 0 0" xyz="0 0 0"/>
 			<geometry>
-				<mesh filename="package://denso_cobotta_descriptions/cobotta_description/J6.dae" scale="1 1 1"/>
-			</geometry>
-		</visual>
-		<collision>
-			<origin rpy="0 0 0" xyz="0 0 0"/>
-			<geometry>
-				<mesh filename="package://denso_cobotta_descriptions/cobotta_description/J6.dae" scale="1 1 1"/>
+				<mesh filename="package://denso_cobotta_descriptions/cobotta_description/J6.dae" scale="${scale} ${scale} ${scale}"/>
+			</geometry>
+		</visual>
+		<collision>
+			<origin rpy="0 0 0" xyz="0 0 0"/>
+			<geometry>
+				<mesh filename="package://denso_cobotta_descriptions/cobotta_description/J6.dae" scale="${scale} ${scale} ${scale}"/>
 			</geometry>
 		</collision>
@@ -250,5 +251,5 @@
 		<parent link="J5"/>
 		<child link="J6"/>
-		<origin rpy="0.000000 0.000000 0.000000" xyz="0.000000 -0.044500 0.042000" />
+		<origin rpy="0.000000 0.000000 0.000000" xyz="0.000000 ${-0.044500*scale} ${0.042000*scale}" />
 		<axis xyz="-0.000000 -0.000000 1.000000" />
 		<limit effort="10" lower="-2.96706" upper="2.96706" velocity="1.1093312725676" />
@@ -266,5 +267,6 @@
 	</transmission>
 	<xacro:if value="${gripper_type != 'none'}">
-		<xacro:include filename="$(find denso_cobotta_descriptions)/cobotta_description/${gripper_type}.urdf.xacro" />
+		<xacro:include filename="$(find assembly_urdf_description)/urdf/${gripper_type}.xacro" />
+		<!-- <xacro:include filename="$(find denso_cobotta_descriptions)/cobotta_description/${gripper_type}.urdf.xacro" /> -->
 	</xacro:if>
 </robot>

Commit message: support gripper-ntlab

File: denso_cobotta_descriptions/cobotta_description/cobotta.urdf.xacro (robot description, xacro)
@@ -6,14 +6,15 @@
 		NOTE: These are roughly estimated values.
 	-->
+	<xacro:property name="mass_adjust" value="1" />
 	<xacro:property name="scale" value ="0.8" />
 	<xacro:property name="joint_damping" value="0.001" />
 	<xacro:property name="joint_friction" value="0.61" />
 	<xacro:property name="base_mass" value="1.4" />
-	<xacro:property name="J1_mass" value="1.29" />
-	<xacro:property name="J2_mass" value="0.39" />
-	<xacro:property name="J3_mass" value="0.35" />
-	<xacro:property name="J4_mass" value="0.35" />
-	<xacro:property name="J5_mass" value="0.19" />
-	<xacro:property name="J6_mass" value="0.03" />
+	<xacro:property name="J1_mass" value="${1.29*mass_adjust}" />
+	<xacro:property name="J2_mass" value="${0.39*mass_adjust}" />
+	<xacro:property name="J3_mass" value="${0.35*mass_adjust}" />
+	<xacro:property name="J4_mass" value="${0.35*mass_adjust}" />
+	<xacro:property name="J5_mass" value="${0.19*mass_adjust}" />
+	<xacro:property name="J6_mass" value="${0.03*mass_adjust}" />
 	<!-- Macro for calculating inertial matrix-->
 	<xacro:macro name="inertia_macro" params="radius height mass *origin">
@@ -267,5 +268,5 @@
 	</transmission>
 	<xacro:if value="${gripper_type != 'none'}">
-		<xacro:include filename="$(find assembly_urdf_description)/urdf/${gripper_type}.xacro" />
+		<xacro:include filename="$(find gripper_ntlab_description)/urdf/${gripper_type}.xacro" />
 		<!-- <xacro:include filename="$(find denso_cobotta_descriptions)/cobotta_description/${gripper_type}.urdf.xacro" /> -->
 	</xacro:if>

File: denso_cobotta_moveit_config/config/cobotta.srdf.xacro (robot description, xacro)
@@ -30,4 +30,7 @@
         <joint name="joint_6" />
     </group>
+    <xacro:if value="${gripper_type == 'gripper_ntlab'}">
+        <xacro:include filename="$(find denso_cobotta_moveit_config)/config/gripper_ntlab.srdf.xacro" />
+    </xacro:if>
     <xacro:if value="${gripper_type == 'parallel'}">
         <xacro:include filename="$(find denso_cobotta_moveit_config)/config/parallel.srdf.xacro" />

Commit message: activate controller for gripper, bring back scale to default

File: denso_cobotta_descriptions/cobotta_description/cobotta.urdf.xacro (robot description, xacro)
@@ -7,5 +7,5 @@
 	-->
 	<xacro:property name="mass_adjust" value="1" />
-	<xacro:property name="scale" value ="0.8" />
+	<xacro:property name="scale" value ="1" />
 	<xacro:property name="joint_damping" value="0.001" />
 	<xacro:property name="joint_friction" value="0.61" />
